File: hardware/SignBuddy_Eagle/SignBuddy Main Board Schematic.sch (EAGLE design)
At the start: 45 parts, among them U1 STM32L053C8T6D, U2 NCP115ASN330T2G

Commit message: Add status led and adc test point
Parts:
- added ADC_TP: TPB1,27, testpad:TPB1,27
- added LED1, LED2: (no value), led:LEDCHIP-LED0603
- added R23, R24: 1.5k, SparkFun-Resistors:1.5KOHM-0603-1/10W-1%
Connections:
- new net LED: LED2.A, U1A.PA8
- new net N$17: LED1.C, R23.2
- new net N$3: LED2.C, R24.2
- net +3V3: now also LED1.A
- net ADC_EXTRA: now also ADC_TP.TP
- net GND: now also R23.1, R24.1
Other:
- note added: "Status LED"
