File: hardware/SignBuddy_Eagle/SignBuddy Main Board Schematic.sch (EAGLE design)
At the start: 42 parts, among them U1 STM32L053C8T6D, U2 NCP115ASN330T2G

Commit message: board done
Parts:
- added 3V3_TP, GND_TP, VBAT_TP: TPB1,27, testpad:TPB1,27
Connections:
- removed net N$3: C6.1, U2.OUT
- removed net RESET: JP1.4
- net +3V3: now also 3V3_TP.TP, C6.1, U2.OUT
- net GND: now also GND_TP.TP
- net NRST: now also JP1.4
- net VBAT: now also VBAT_TP.TP
Changed lines of the file:
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@@
 <part name="JP2" library="pinhead" library_urn="urn:adsk.eagle:library:325" deviceset="PINHD-1X2" device="" package3d_urn="urn:adsk.eagle:package:22435/2"/>
 <part name="GND13" library="supply1" library_urn="urn:adsk.eagle:library:371" deviceset="GND" device=""/>
+<part name="VBAT_TP" library="testpad" library_urn="urn:adsk.eagle:library:385" deviceset="TP" device="B1,27" package3d_urn="urn:adsk.eagle:package:27944/2"/>
+<part name="3V3_TP" library="testpad" library_urn="urn:adsk.eagle:library:385" deviceset="TP" device="B1,27" package3d_urn="urn:adsk.eagle:package:27944/2"/>
+<part name="GND_TP" library="testpad" library_urn="urn:adsk.eagle:library:385" deviceset="TP" device="B1,27" package3d_urn="urn:adsk.eagle:package:27944/2"/>
+<part name="+3V13" library="supply1" library_urn="urn:adsk.eagle:library:371" deviceset="+3V3" device=""/>
 </parts>
 <sheets>
@@
 <label x="76.2" y="25.4" size="1.778" layer="95"/>
 </segment>
+<segment>
+<pinref part="JP1" gate="A" pin="4"/>
+<wire x1="-73.66" y1="-73.66" x2="-99.06" y2="-73.66" width="0.1524" layer="91"/>
+<label x="-99.06" y="-73.66" size="1.778" layer="95"/>
+</segment>
 </net>
 <net name="BOOT0_LOW" class="0">
@@
 <wire x1="114.3" y1="35.56" x2="114.3" y2="12.7" width="0.1524" layer="91"/>
 <label x="114.3" y="12.7" size="1.778" layer="95" rot="R90"/>
-</segment>
-</net>
-<net name="RESET" class="0">
-<segment>
-<pinref part="JP1" gate="A" pin="4"/>
-<wire x1="-73.66" y1="-73.66" x2="-99.06" y2="-73.66" width="0.1524" layer="91"/>
-<label x="-99.06" y="-73.66" size="1.778" layer="95"/>
 </segment>
 </net>
@@
 <attribute name="VALUE" x="45.72" y="43.18" size="1.778" layer="96"/>
 </instance>
+<instance part="VBAT_TP" gate="G$1" x="-106.68" y="53.34" smashed="yes">
+<attribute name="NAME" x="-107.95" y="54.61" size="1.778" layer="95"/>
+<attribute name="TP_SIGNAL_NAME" x="-105.41" y="52.07" size="1.778" layer="97"/>
+</instance>
+<instance part="3V3_TP" gate="G$1" x="-35.56" y="50.8" smashed="yes">
+<attribute name="NAME" x="-36.83" y="52.07" size="1.778" layer="95"/>
+<attribute name="TP_SIGNAL_NAME" x="-34.29" y="49.53" size="1.778" layer="97"/>
+</instance>
+<instance part="GND_TP" gate="G$1" x="-93.98" y="50.8" smashed="yes">
+<attribute name="NAME" x="-95.25" y="52.07" size="1.778" layer="95"/>
+<attribute name="TP_SIGNAL_NAME" x="-92.71" y="49.53" size="1.778" layer="97"/>
+</instance>
+<instance part="+3V13" gate="G$1" x="-27.94" y="58.42" smashed="yes">
+<attribute name="VALUE" x="-27.94" y="58.42" size="1.778" layer="96"/>
+</instance>
 </instances>
 <busses>
@@
 <pinref part="U2" gate="A" pin="EN"/>
 <wire x1="-86.36" y1="50.8" x2="-104.14" y2="50.8" width="0.1524" layer="91"/>
-<wire x1="-104.14" y1="50.8" x2="-114.3" y2="50.8" width="0.1524" layer="91"/>
+<wire x1="-104.14" y1="50.8" x2="-106.68" y2="50.8" width="0.1524" layer="91"/>
+<wire x1="-106.68" y1="50.8" x2="-114.3" y2="50.8" width="0.1524" layer="91"/>
 <wire x1="-81.28" y1="45.72" x2="-86.36" y2="45.72" width="0.1524" layer="91"/>
 <wire x1="-86.36" y1="45.72" x2="-86.36" y2="50.8" width="0.1524" layer="91"/>
@@
 <pinref part="C7" gate="G$1" pin="1"/>
 <junction x="-104.14" y="50.8"/>
+<pinref part="VBAT_TP" gate="G$1" pin="TP"/>
+<junction x="-106.68" y="50.8"/>
 </segment>
 <segment>
@@
 <segment>
 <pinref part="U2" gate="A" pin="GND"/>
-<wire x1="-81.28" y1="48.26" x2="-96.52" y2="48.26" width="0.1524" layer="91"/>
+<wire x1="-81.28" y1="48.26" x2="-93.98" y2="48.26" width="0.1524" layer="91"/>
+<wire x1="-93.98" y1="48.26" x2="-96.52" y2="48.26" width="0.1524" layer="91"/>
 <wire x1="-96.52" y1="48.26" x2="-96.52" y2="43.18" width="0.1524" layer="91"/>
 <pinref part="GND9" gate="1" pin="GND"/>
@@
 <wire x1="-104.14" y1="43.18" x2="-96.52" y2="43.18" width="0.1524" layer="91"/>
 <junction x="-96.52" y="43.18"/>
+<pinref part="GND_TP" gate="G$1" pin="TP"/>
+<junction x="-93.98" y="48.26"/>
 </segment>
 <segment>
@@
 <wire x1="48.26" y1="53.34" x2="48.26" y2="48.26" width="0.1524" layer="91"/>
 <pinref part="GND13" gate="1" pin="GND"/>
-</segment>
-</net>
-<net name="N$3" class="0">
-<segment>
-<pinref part="U2" gate="A" pin="OUT"/>
-<wire x1="-45.72" y1="48.26" x2="-27.94" y2="48.26" width="0.1524" layer="91"/>
-<pinref part="C6" gate="G$1" pin="1"/>
 </segment>
 </net>
@@
 </segment>
 </net>
+<net name="+3V3" class="0">
+<segment>
+<pinref part="U2" gate="A" pin="OUT"/>
+<wire x1="-45.72" y1="48.26" x2="-35.56" y2="48.26" width="0.1524" layer="91"/>
+<pinref part="C6" gate="G$1" pin="1"/>
+<pinref part="3V3_TP" gate="G$1" pin="TP"/>
+<wire x1="-35.56" y1="48.26" x2="-27.94" y2="48.26" width="0.1524" layer="91"/>
+<junction x="-35.56" y="48.26"/>
+<pinref part="+3V13" gate="G$1" pin="+3V3"/>
+<wire x1="-27.94" y1="48.26" x2="-27.94" y2="55.88" width="0.1524" layer="91"/>
+<junction x="-27.94" y="48.26"/>
+</segment>
+</net>

Commit message: Add status led and adc test point (#124)
* Add status led and adc test point

* fixes

Co-authored-by: Adam Bujak <adamjbujak@gmail.com>
Parts:
- added ADC_TP: TPB1,27, testpad:TPB1,27
- added LED1, LED2: (no value), led:LEDCHIP-LED0603
- added R23, R24: 1k, SparkFun-Resistors:1.5KOHM-0603-1/10W-1%
Connections:
- new net LED: LED2.A, U1A.PA8
- new net N$17: LED1.C, R23.2
- new net N$3: LED2.C, R24.2
- net +3V3: now also LED1.A
- net ADC_EXTRA: now also ADC_TP.TP
- net GND: now also R23.1, R24.1
Other:
- note added: "LEDs"
Changed lines of the file:
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@@
 <part name="GND_TP" library="testpad" library_urn="urn:adsk.eagle:library:385" deviceset="TP" device="B1,27" package3d_urn="urn:adsk.eagle:package:27944/2"/>
 <part name="+3V13" library="supply1" library_urn="urn:adsk.eagle:library:371" deviceset="+3V3" device=""/>
+<part name="R23" library="SparkFun-Resistors" library_urn="urn:adsk.eagle:library:532" deviceset="1.5KOHM" device="-0603-1/10W-1%" package3d_urn="urn:adsk.eagle:package:39650/1" value="1k"/>
+<part name="R24" library="SparkFun-Resistors" library_urn="urn:adsk.eagle:library:532" deviceset="1.5KOHM" device="-0603-1/10W-1%" package3d_urn="urn:adsk.eagle:package:39650/1" value="1k"/>
+<part name="GND14" library="supply1" library_urn="urn:adsk.eagle:library:371" deviceset="GND" device=""/>
+<part name="GND15" library="supply1" library_urn="urn:adsk.eagle:library:371" deviceset="GND" device=""/>
+<part name="ADC_TP" library="testpad" library_urn="urn:adsk.eagle:library:385" deviceset="TP" device="B1,27" package3d_urn="urn:adsk.eagle:package:27944/2"/>
+<part name="LED1" library="led" library_urn="urn:adsk.eagle:library:259" deviceset="LED" device="CHIP-LED0603" package3d_urn="urn:adsk.eagle:package:15819/3"/>
+<part name="LED2" library="led" library_urn="urn:adsk.eagle:library:259" deviceset="LED" device="CHIP-LED0603" package3d_urn="urn:adsk.eagle:package:15819/3"/>
 </parts>
 <sheets>
@@
 </instance>
 <instance part="U$2" gate="G$1" x="-2.54" y="-73.66" smashed="yes"/>
+<instance part="ADC_TP" gate="G$1" x="-22.86" y="5.08" smashed="yes">
+<attribute name="NAME" x="-24.13" y="6.35" size="1.778" layer="95"/>
+<attribute name="TP_SIGNAL_NAME" x="-21.59" y="3.81" size="1.778" layer="97"/>
+</instance>
 </instances>
 <busses>
@@
 <segment>
 <pinref part="U1" gate="A" pin="PB1"/>
-<wire x1="10.16" y1="2.54" x2="-7.62" y2="2.54" width="0.1524" layer="91"/>
+<wire x1="10.16" y1="2.54" x2="-22.86" y2="2.54" width="0.1524" layer="91"/>
 <label x="-7.62" y="2.54" size="1.27" layer="95"/>
+<pinref part="ADC_TP" gate="G$1" pin="TP"/>
 </segment>
 </net>
@@
 </segment>
 </net>
+<net name="LED" class="0">
+<segment>
+<pinref part="U1" gate="A" pin="PA8"/>
+<wire x1="10.16" y1="27.94" x2="-7.62" y2="27.94" width="0.1524" layer="91"/>
+<label x="-7.62" y="27.94" size="1.27" layer="95"/>
+</segment>
+</net>
 </nets>
 </sheet>
@@
 <text x="-81.28" y="7.62" size="3.81" layer="91">Battery Connector</text>
 <text x="48.26" y="81.28" size="3.81" layer="91">Log UART</text>
+<text x="50.8" y="10.16" size="3.81" layer="91">LEDs</text>
 </plain>
 <instances>
@@
 <instance part="+3V13" gate="G$1" x="-27.94" y="58.42" smashed="yes">
 <attribute name="VALUE" x="-27.94" y="58.42" size="1.778" layer="96"/>
+</instance>
+<instance part="R23" gate="G$1" x="27.94" y="-7.62" smashed="yes" rot="R90">
+<attribute name="NAME" x="26.416" y="-7.62" size="1.778" layer="95" font="vector" rot="R90" align="bottom-center"/>
+<attribute name="VALUE" x="29.464" y="-7.62" size="1.778" layer="96" font="vector" rot="R90" align="top-center"/>
+</instance>
+<instance part="R24" gate="G$1" x="71.12" y="-7.62" smashed="yes" rot="R90">
+<attribute name="NAME" x="69.596" y="-7.62" size="1.778" layer="95" font="vector" rot="R90" align="bottom-center"/>
+<attribute name="VALUE" x="72.644" y="-7.62" size="1.778" layer="96" font="vector" rot="R90" align="top-center"/>
+</instance>
+<instance part="GND14" gate="1" x="27.94" y="-15.24" smashed="yes">
+<attribute name="VALUE" x="25.4" y="-17.78" size="1.778" layer="96"/>
+</instance>
+<instance part="GND15" gate="1" x="71.12" y="-15.24" smashed="yes">
+<attribute name="VALUE" x="68.58" y="-17.78" size="1.778" layer="96"/>
+</instance>
+<instance part="LED1" gate="G$1" x="40.64" y="-2.54" smashed="yes" rot="R270">
+<attribute name="NAME" x="36.068" y="-6.096" size="1.778" layer="95"/>
+<attribute name="VALUE" x="36.068" y="-8.255" size="1.778" layer="96"/>
+</instance>
+<instance part="LED2" gate="G$1" x="83.82" y="-2.54" smashed="yes" rot="R270">
+<attribute name="NAME" x="79.248" y="-6.096" size="1.778" layer="95"/>
+<attribute name="VALUE" x="79.248" y="-8.255" size="1.778" layer="96"/>
 </instance>
 </instances>
@@
 <pinref part="GND13" gate="1" pin="GND"/>
 </segment>
+<segment>
+<pinref part="R23" gate="G$1" pin="1"/>
+<pinref part="GND14" gate="1" pin="GND"/>
+</segment>
+<segment>
+<pinref part="R24" gate="G$1" pin="1"/>
+<pinref part="GND15" gate="1" pin="GND"/>
+</segment>
 </net>
 <net name="N$2" class="0">
@@
 <wire x1="-2.54" y1="-27.94" x2="-121.92" y2="-27.94" width="0.1524" layer="91" style="longdash"/>
 <wire x1="-2.54" y1="17.78" x2="127" y2="17.78" width="0.1524" layer="91" style="longdash"/>
+<wire x1="-2.54" y1="-27.94" x2="127" y2="-27.94" width="0.1524" layer="91" style="longdash"/>
 </segment>
 </net>
@@
 <wire x1="-27.94" y1="48.26" x2="-27.94" y2="55.88" width="0.1524" layer="91"/>
 <junction x="-27.94" y="48.26"/>
-</segment>
-</net>
+<wire x1="-27.94" y1="48.26" x2="-27.94" y2="55.88" width="0.1524" layer="91"/>
+</segment>
+<segment>
+<wire x1="43.18" y1="-2.54" x2="50.8" y2="-2.54" width="0.1524" layer="91"/>
+<label x="48.26" y="0" size="1.778" layer="95"/>
+<pinref part="LED1" gate="G$1" pin="A"/>
+</segment>
+</net>
+<net name="N$3" class="0">
+<segment>
+<pinref part="R24" gate="G$1" pin="2"/>
+<wire x1="78.74" y1="-2.54" x2="71.12" y2="-2.54" width="0.1524" layer="91"/>
+<pinref part="LED2" gate="G$1" pin="C"/>
+</segment>
+</net>
+<net name="N$17" class="0">
+<segment>
+<pinref part="R23" gate="G$1" pin="2"/>
+<wire x1="35.56" y1="-2.54" x2="27.94" y2="-2.54" width="0.1524" layer="91"/>
+<pinref part="LED1" gate="G$1" pin="C"/>
+</segment>
+</net>
+<net name="LED" class="0">
+<segment>
+<wire x1="88.9" y1="-2.54" x2="96.52" y2="-2.54" width="0.1524" layer="91"/>
+<label x="96.52" y="-2.54" size="1.778" layer="95"/>
+<wire x1="96.52" y1="-2.54" x2="99.06" y2="-2.54" width="0.1524" layer="91"/>
+<wire x1="86.36" y1="-2.54" x2="88.9" y2="-2.54" width="0.1524" layer="91"/>
+<pinref part="LED2" gate="G$1" pin="A"/>
+</segment>
+</net>

Commit message: small position adjustments
Changed lines of the file:
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@@
 <junction x="-35.56" y="48.26"/>
 <pinref part="+3V13" gate="G$1" pin="+3V3"/>
-<wire x1="-27.94" y1="48.26" x2="-27.94" y2="55.88" width="0.1524" layer="91"/>
 <junction x="-27.94" y="48.26"/>
 <wire x1="-27.94" y1="48.26" x2="-27.94" y2="55.88" width="0.1524" layer="91"/>
