File: hardware/SignBuddy_Eagle/SignBuddy Main Board Schematic.brd (EAGLE design)
At the start: 54.1 x 47.5 mm, 45 parts, among them U1 STM32L053C8T6D, U2 NCP115ASN330T2G

Commit message: Add status led and adc test point
Parts:
- added ADC_TP: TPB1,27, testpad:B1,27
- added LED1, LED2: (no value), led:CHIP-LED0603
- added R23, R24: 1.5k, SparkFun-Resistors:0603
Connections:
- new net LED: LED2.A, U1.29
- new net N$17: LED1.C, R23.2
- new net N$3: LED2.C, R24.2
- net +3V3: now also LED1.A
- net ADC_EXTRA: now also ADC_TP.TP
- net GND: now also R23.1, R24.1
Routing:
- net LED: track 0.00 -> 14.4 mm, vias 0 -> 4
- net ADC_EXTRA: track 0.00 -> 8.20 mm
- net +3V3: track 26.2 -> 30.8 mm
- net N$3: track 0.00 -> 2.97 mm
- net N$17: track 0.00 -> 2.72 mm
Changed lines of the file:
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@@
 <drawing>
 <settings>
-<setting alwaysvectorfont="no"/>
+<setting alwaysvectorfont="yes"/>
 <setting verticaltext="up"/>
 </settings>
@@
 <layer number="43" name="vRestrict" color="2" fill="10" visible="yes" active="yes"/>
 <layer number="44" name="Drills" color="7" fill="1" visible="no" active="yes"/>
-<layer number="45" name="Holes" color="7" fill="1" visible="no" active="yes"/>
+<layer number="45" name="Holes" color="7" fill="1" visible="yes" active="yes"/>
 <layer number="46" name="Milling" color="3" fill="1" visible="no" active="yes"/>
 <layer number="47" name="Measures" color="7" fill="1" visible="no" active="yes"/>
@@
 <attribute name="VALUE" x="32.639" y="7.874" size="0.0254" layer="28" rot="MR0"/>
 </element>
+<element name="R23" library="SparkFun-Resistors" library_urn="urn:adsk.eagle:library:532" package="0603" package3d_urn="urn:adsk.eagle:package:39650/1" value="1.5k" x="33.02" y="1.016" smashed="yes">
+<attribute name="NAME" x="33.02" y="1.778" size="0.6096" layer="25" font="vector" ratio="20" align="bottom-center"/>
+<attribute name="PROD_ID" value="RES-08306" x="33.02" y="1.016" size="1.778" layer="27" display="off"/>
+<attribute name="VALUE" x="33.02" y="0.254" size="0.6096" layer="27" font="vector" ratio="20" align="top-center"/>
+</element>
+<element name="R24" library="SparkFun-Resistors" library_urn="urn:adsk.eagle:library:532" package="0603" package3d_urn="urn:adsk.eagle:package:39650/1" value="1.5k" x="46.228" y="1.016" smashed="yes">
+<attribute name="NAME" x="46.228" y="1.778" size="0.6096" layer="25" font="vector" ratio="20" align="bottom-center"/>
+<attribute name="PROD_ID" value="RES-08306" x="46.228" y="1.016" size="1.778" layer="27" display="off"/>
+<attribute name="VALUE" x="46.228" y="0.254" size="0.6096" layer="27" font="vector" ratio="20" align="top-center"/>
+</element>
+<element name="ADC_TP" library="testpad" library_urn="urn:adsk.eagle:library:385" package="B1,27" package3d_urn="urn:adsk.eagle:package:27944/2" value="TPB1,27" x="41.148" y="1.27" smashed="yes">
+<attribute name="NAME" x="40.513" y="2.286" size="1.27" layer="25" ratio="10"/>
+<attribute name="POPULARITY" value="19" x="41.148" y="1.27" size="1.778" layer="27" display="off"/>
+<attribute name="TP_SIGNAL_NAME" value="" x="41.148" y="1.27" size="1.778" layer="27" display="off"/>
+<attribute name="VALUE" x="40.513" y="0.508" size="0.0254" layer="27"/>
+</element>
+<element name="LED1" library="led" library_urn="urn:adsk.eagle:library:259" package="CHIP-LED0603" package3d_urn="urn:adsk.eagle:package:15819/3" value="" x="37.338" y="1.016" smashed="yes" rot="R90">
+<attribute name="NAME" x="37.973" y="0.381" size="1.27" layer="25" rot="R180"/>
+<attribute name="POPULARITY" value="26" x="37.338" y="1.016" size="1.778" layer="27" rot="R90" display="off"/>
+<attribute name="VALUE" x="37.973" y="2.921" size="1.27" layer="27" rot="R180"/>
+</element>
+<element name="LED2" library="led" library_urn="urn:adsk.eagle:library:259" package="CHIP-LED0603" package3d_urn="urn:adsk.eagle:package:15819/3" value="" x="50.8" y="1.016" smashed="yes" rot="R90">
+<attribute name="NAME" x="51.435" y="0.381" size="1.27" layer="25" rot="R180"/>
+<attribute name="POPULARITY" value="26" x="50.8" y="1.016" size="1.778" layer="27" rot="R90" display="off"/>
+<attribute name="VALUE" x="51.435" y="2.921" size="1.27" layer="27" rot="R180"/>
+</element>
 </elements>
 <signals>
@@
 <signal name="ADC_EXTRA">
 <contactref element="U1" pad="19"/>
+<contactref element="ADC_TP" pad="TP"/>
+<wire x1="42.564" y1="8.882" x2="42.564" y2="5.988" width="0.1524" layer="1"/>
+<wire x1="42.564" y1="5.988" x2="41.91" y2="5.334" width="0.1524" layer="1"/>
+<wire x1="41.91" y1="2.032" x2="41.148" y2="1.27" width="0.1524" layer="1"/>
+<wire x1="41.91" y1="5.334" x2="41.91" y2="2.032" width="0.1524" layer="1"/>
 </signal>
 <signal name="TSC_G4_E2">
@@
 <wire x1="48.768" y1="38.354" x2="48.768" y2="42.3" width="0.4064" layer="16"/>
 <wire x1="48.768" y1="42.3" x2="48.556" y2="42.512" width="0.4064" layer="16"/>
+<contactref element="R23" pad="1"/>
+<contactref element="R24" pad="1"/>
+<wire x1="45.378" y1="1.016" x2="32.17" y2="1.016" width="0" layer="19" extent="1-1"/>
+<wire x1="51.308" y1="3.81" x2="45.378" y2="1.016" width="0" layer="19" extent="1-1"/>
 </signal>
 <signal name="BOOT0">
@@
 <wire x1="9.0126" y1="21.082" x2="9.5206" y2="20.574" width="0.3048" layer="1"/>
 <wire x1="9.5206" y1="20.574" x2="10.072" y2="20.574" width="0.3048" layer="1"/>
+<contactref element="LED1" pad="A"/>
+<wire x1="38.088" y1="1.016" x2="38.088" y2="2.044" width="0.1524" layer="1"/>
+<wire x1="38.088" y1="2.044" x2="35.56" y2="4.572" width="0.1524" layer="1"/>
+<wire x1="45.125" y1="30.06" x2="38.396" y2="42.512" width="0" layer="19" extent="1-1"/>
+<wire x1="48.28" y1="22.116" x2="45.125" y2="30.06" width="0" layer="19" extent="1-1"/>
+<wire x1="46.564" y1="15.882" x2="48.28" y2="22.116" width="0" layer="19" extent="1-1"/>
+<wire x1="39.564" y1="17.382" x2="46.564" y2="15.882" width="0" layer="19" extent="1-1"/>
+<wire x1="38.064" y1="15.882" x2="39.564" y2="17.382" width="0" layer="19" extent="1-1"/>
+<wire x1="34.604" y1="16.422" x2="38.064" y2="15.882" width="0" layer="19" extent="1-1"/>
+<wire x1="34.526" y1="20.642" x2="34.604" y2="16.422" width="0" layer="19" extent="1-1"/>
+<wire x1="29.972" y1="10.668" x2="34.798" y2="12.192" width="0" layer="19" extent="16-16"/>
+<wire x1="28.00985" y1="13.142" x2="29.972" y2="10.668" width="0" layer="19" extent="1-16"/>
+<wire x1="35.56" y1="4.572" x2="29.806" y2="8.128" width="0" layer="19" extent="1-1"/>
+<wire x1="45.064" y1="8.882" x2="46.564" y2="15.882" width="0" layer="19" extent="1-1"/>
+<wire x1="51.112" y1="6.516" x2="45.064" y2="8.882" width="0" layer="19" extent="1-1"/>
+<wire x1="14.224" y1="15.748" x2="26.2934" y2="15.99500625" width="0" layer="19" extent="1-1"/>
+<wire x1="11.772" y1="16.002" x2="11.772" y2="13.716" width="0" layer="19" extent="1-1"/>
+<wire x1="11.772" y1="18.288" x2="11.772" y2="16.002" width="0" layer="19" extent="1-1"/>
+<wire x1="10.072" y1="22.86" x2="9.0126" y2="21.082" width="0" layer="19" extent="1-1"/>
+<wire x1="12.7" y1="4.572" x2="11.772" y2="13.716" width="0" layer="19" extent="1-1"/>
 </signal>
 <signal name="NRST">
@@
 <wire x1="20.828" y1="40.64" x2="20.828" y2="41.656" width="0.1524" layer="1"/>
 </signal>
+<signal name="N$3">
+<contactref element="R24" pad="2"/>
+<contactref element="LED2" pad="C"/>
+<wire x1="50.05" y1="1.016" x2="47.078" y2="1.016" width="0.1524" layer="1"/>
+</signal>
+<signal name="N$17">
+<contactref element="R23" pad="2"/>
+<contactref element="LED1" pad="C"/>
+<wire x1="36.588" y1="1.016" x2="33.87" y2="1.016" width="0.1524" layer="1"/>
+</signal>
+<signal name="LED">
+<contactref element="U1" pad="29"/>
+<contactref element="LED2" pad="A"/>
+<wire x1="46.564" y1="12.382" x2="47.816" y2="12.382" width="0.1524" layer="1"/>
+<wire x1="47.816" y1="12.382" x2="48.26" y2="11.938" width="0.1524" layer="1"/>
+<via x="48.26" y="11.938" extent="1-16" drill="0.35"/>
+<wire x1="48.26" y1="11.938" x2="48.26" y2="8.128" width="0.1524" layer="16"/>
+<via x="48.26" y="8.128" extent="1-16" drill="0.35"/>
+<wire x1="48.26" y1="8.128" x2="49.53" y2="6.858" width="0.1524" layer="1"/>
+<wire x1="49.53" y1="6.858" x2="49.53" y2="4.318" width="0.1524" layer="1"/>
+<via x="49.53" y="4.318" extent="1-16" drill="0.35"/>
+<wire x1="49.53" y1="4.318" x2="51.816" y2="2.032" width="0.1524" layer="16"/>
+<via x="51.816" y="2.032" extent="1-16" drill="0.35"/>
+<wire x1="51.816" y1="2.032" x2="51.816" y2="1.282" width="0.1524" layer="1"/>
+<wire x1="51.816" y1="1.282" x2="51.55" y2="1.016" width="0.1524" layer="1"/>
+</signal>
 </signals>

Commit message: fixes
Parts:
- R23, R24: value 1.5k -> 1k
- moved C4 0.57 mm to (51.4, 6.17)
- moved VBAT_TP 0.36 mm to (25.1, 15.5)
- moved 3V3_TP 0.25 mm to (30.0, 10.9)
Routing:
- net +3V3: track 30.8 -> 58.5 mm, vias 8 -> 10
- net GND: track 107.1 -> 112.9 mm, vias 19 -> 21
- net LED: track 14.4 -> 19.3 mm, vias 4 -> 2
- net TSC_G6_E1: track 81.1 -> 79.4 mm
- net LOG_UART_TX: track 78.1 -> 78.6 mm
